Commit message: 增加urdf

File: src/r2bot_description/urdf/r2bot.urdf (robot description, URDF)
Before this commit: robot roverbot, 3 links, 2 joints
Links:
- link base_link: geometry visual box size=0.65 0.65 0.18
Joints:
- joint base_joint: origin xyz=0.0 0.0 0.0 rpy=0 0 0 -> xyz=0.0 0.0 0.09 rpy=0 0 0
- joint laser_joint: origin xyz=-0.05 0 0.144 rpy=0 0 0 -> xyz=0.325 0.0 0.13 rpy=0 0 0

Commit message: r2更新雷达定位

File: src/r2bot_description/urdf/r2bot.urdf (robot description, URDF)
Before this commit: robot r2bot, 3 links, 2 joints
Links:
- added link camera_color_frame
- added link camera_color_optical_frame
- added link camera_depth_frame
- added link camera_depth_optical_frame
- added link camera_link; visual box size=0.09 0.03 0.025
Joints:
- added joint camera_color_joint: type fixed, parent camera_link, child camera_color_frame, origin xyz=0 0 0 rpy=0 0 0
- added joint camera_color_optical_joint: type fixed, parent camera_color_frame, child camera_color_optical_frame, origin xyz=0 0 0 rpy=-1.57079632679 0 -1.57079632679
- added joint camera_depth_joint: type fixed, parent camera_link, child camera_depth_frame, origin xyz=0 0 0 rpy=0 0 0
- added joint camera_depth_optical_joint: type fixed, parent camera_depth_frame, child camera_depth_optical_frame, origin xyz=0 0 0 rpy=-1.57079632679 0 -1.57079632679
- added joint camera_joint: type fixed, parent base_link, child camera_link, origin xyz=0.245 0.0 0.235 rpy=0 0 0

Commit message: 更新urdf

File: src/r2bot_description/urdf/r2bot.urdf (robot description, URDF)
Before this commit: robot r2bot, 8 links, 7 joints
Links:
- link base_link: geometry visual box size=0.8 0.73 0.18
Joints:
- joint laser_joint: origin xyz=0.325 0.0 0.13 rpy=0 0 0 -> xyz=0.2 0.135 0.145 rpy=0 0 0
